Commit message: transmissions

File: ur10_e_moveit_config/ur10e_robotiq85/urdf/ur10e_robotiq85_switch.urdf (robot description, URDF)
Before this commit: robot ur10e_robotiq, 20 links, 19 joints
Links:
- added link left_inner_finger_pad; collision box size=0.022 0.00635 0.0375; visual box size=0.022 0.00635 0.05
- link gripper_robotiq_85_left_finger_tip_link: geometry collision mesh filename=package://cable_simulation/meshes/collision/robotiq_arg2f_8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 scale=0.001 0.001 0.001; visual mesh filename=package://cable_simulation/meshes/visual/robotiq_arg2f_85_i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 scale=0.001 0.001 0.001
Joints:
- added joint left_inner_finger_pad_joint: type fixed, parent gripper_robotiq_85_left_finger_tip_link, child left_inner_finger_pad, origin xyz=0.03175 0.0035 0 rpy=0 0 0, axis 0 0 1

Commit message: switch urdfs update

File: ur10_e_moveit_config/ur10e_robotiq85/urdf/ur10e_robotiq85_switch.urdf (robot description, URDF)
Before this commit: robot ur10e_robotiq, 21 links, 20 joints
Links:
- added link right_inner_finger_pad; collision box size=0.022 0.00635 0.05; visual box size=0.022 0.00635 0.05
- link gripper_robotiq_85_right_finger_tip_link: geometry collision mesh filename=package://cable_simulation/meshes/collision/robotiq_arg2f_8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 scale=0.001 0.001 0.001; visual mesh filename=package://cable_simulation/meshes/visual/robotiq_arg2f_85_i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 scale=0.001 0.001 0.001
- link left_inner_finger_pad: geometry collision box size=0.022 0.00635 0.05; visual box size=0.022 0.00635 0.05
Joints:
- added joint right_inner_finger_pad_joint: type fixed, parent gripper_robotiq_85_right_finger_tip_link, child right_inner_finger_pad, origin xyz=0.03175 0.0035 0 rpy=0 0 0, axis 0 0 1

Commit message: switch

File: ur10_e_moveit_config/ur10e_robotiq85/urdf/ur10e_robotiq85_switch.urdf (robot description, URDF)
Before this commit: robot ur10e_robotiq, 22 links, 21 joints
Joints:
- joint left_inner_finger_pad_joint: origin xyz=0.03175 0.0035 0 rpy=0 0 0 -> xyz=-0.003536 0.0035 0 rpy=0 0 0

Commit message: position switch flange urdf update

File: ur10_e_moveit_config/ur10e_robotiq85/urdf/ur10e_robotiq85_switch.urdf (robot description, URDF)
Before this commit: robot ur10e_robotiq_switch, 22 links, 21 joints
Joints:
- joint left_inner_finger_pad_joint: origin xyz=-0.003536 0.0035 0 rpy=0 0 0 -> xyz=0.03175 0.0035 0 rpy=0 0 0

File: ur10_e_moveit_config/ur10e_robotiq_85/urdf1/ur10e_robotiq85_flange.urdf (robot description, URDF)
Before this commit: robot ur10e_robotiq85_flange, 21 links, 20 joints
Links:
- link flange_link: geometry collision mesh filename=package://ur10e_85_flange_moveit/flange/adapter.stl scale=0.025 0.025 0.025; visual mesh filename=package://ur10e_85_flange_moveit/flange/adapter.stl scale=0.025 0.025 0.025
Joints:
- joint flange-robotiq_85_base_joint: origin xyz=0 0 0.025 rpy=0 -1.57079632679 1.57079632679 -> xyz=0 0 0.08 rpy=0 -1.57079632679 1.57079632679
- joint robot_tool0-flange_joint: origin xyz=0 0 0.025 rpy=0 0 0 -> xyz=0 0 0.0 rpy=0 0 0
