Commit message: flange

File: ur10_e_moveit_config/ur10e_robotiq_85/urdf1/ur10e_robotiq85_flange.xacro (robot description, xacro)
@@ -1,3 +1,3 @@
-<robot name="ur10e_robotiq" xmlns:xacro="http://wiki.ros.org/xacro">
+<robot name="ur10e_robotiq85_flange" xmlns:xacro="http://wiki.ros.org/xacro">
     <!-- include macros for UR10 and the 2f_85 gripper -->
     <xacro:include filename="$(find ur_e_description)/urdf/ur10e.urdf.xacro" />
@@ -9,8 +9,21 @@
     <xacro:ur10e_robot prefix="${prefix}robot_" joint_limited="true"/>
     <xacro:robotiq_85_gripper prefix="${prefix}gripper_" />
+  <!-- include camera flange -->
+  <joint name="${prefix}robot_tool0-${prefix}flange_joint" type="fixed">
+    <origin xyz="0 0 0.025" rpy="0 0 0" />
+    <parent link="${prefix}robot_tool0" />
+    <child link="${prefix}flange_link" />
+  </joint>
+  <link name="flange_link">
+    <visual>
+      <geometry>
+        <cylinder length="0.05" radius="0.05"/>
+      </geometry>
+    </visual>
+  </link>
   <!-- attach gripper -->
-  <joint name="${prefix}robot_tool0-${prefix}robotiq_85_base_link" type="fixed">
-    <origin xyz="0 0 0" rpy="0 -${pi/2} ${pi/2}" />
-    <parent link="${prefix}robot_tool0" />
+  <joint name="${prefix}flange-${prefix}robotiq_85_base_joint" type="fixed">
+    <origin xyz="0 0 0.025" rpy="0 -${pi/2} ${pi/2}" />
+    <parent link="${prefix}flange_link" />
     <child link="${prefix}gripper_robotiq_85_base_link" />
   </joint>

Commit message: xacro and urdf clean up

File: ur10_e_moveit_config/ur10e_robotiq_85/urdf1/ur10e_robotiq85_flange.xacro (robot description, xacro)
@@ -1,12 +1,12 @@
 <robot name="ur10e_robotiq85_flange" xmlns:xacro="http://wiki.ros.org/xacro">
-    <!-- include macros for UR10 and the 2f_85 gripper -->
-    <xacro:include filename="$(find ur_e_description)/urdf/ur10e.urdf.xacro" />
-    <xacro:include filename="$(find cable_simulation)/urdf/robotiq_85_gripper.urdf.xacro" />
-    <xacro:arg name="limited" default="true"/>
-    <!-- create the robot + eef combo itself as a macro -->
-    <xacro:macro name="ee_robot" params="prefix">
-    <!-- instantiate UR10e and 2f_85 gripper -->
-    <xacro:ur10e_robot prefix="${prefix}robot_" joint_limited="true"/>
-    <xacro:robotiq_85_gripper prefix="${prefix}gripper_" />
+  <!-- include macros for UR10 and the 2f_85 gripper -->
+  <xacro:include filename="$(find ur_e_description)/urdf/ur10e.urdf.xacro" />
+  <xacro:include filename="$(find cable_simulation)/urdf/robotiq_85_gripper.urdf.xacro" />
+  <xacro:arg name="limited" default="true"/>
+  <!-- create the robot + eef combo itself as a macro -->
+  <xacro:macro name="ee_robot" params="prefix">
+  <!-- instantiate UR10e and 2f_85 gripper -->
+  <xacro:ur10e_robot prefix="${prefix}robot_" joint_limited="true"/>
+  <xacro:robotiq_85_gripper prefix="${prefix}gripper_" />
   <!-- include camera flange -->
   <joint name="${prefix}robot_tool0-${prefix}flange_joint" type="fixed">
@@ -30,9 +30,9 @@
   <!-- define the ur10's position and orientation in the world coordinate system -->
     <link name="world"/>
+    <!-- TODO: check base_link name of robot -->
     <joint name="world_joint" type="fixed">
-    <parent link="world"/>
-    <child link="robot_base_link"/>
-    <!-- TODO: check base_link name of robot -->
-    <origin rpy="0.0 0.0 0.0" xyz="0.0 0.0 0.0"/>
+      <parent link="world"/>
+      <child link="robot_base_link"/>
+      <origin rpy="0.0 0.0 0.0" xyz="0.0 0.0 0.0"/>
     </joint>
  </xacro:macro>
